Commit message: Fix Mismatch component for loading HybridFTController

File: franka_robot.urdf (robot description, URDF)
Before this commit: robot fr3, 14 links, 13 joints
Links:
- added link fr3_link0_accelerometer_bottom
- added link fr3_link0_accelerometer_top
- added link fr3_link1_accelerometer_bottom
- added link fr3_link1_accelerometer_top
- added link fr3_link2_accelerometer_bottom
- added link fr3_link2_accelerometer_top
- added link fr3_link3_accelerometer_bottom
- added link fr3_link3_accelerometer_top
- added link fr3_link4_accelerometer_bottom
- added link fr3_link4_accelerometer_top
- added link fr3_link5_accelerometer_bottom
- added link fr3_link5_accelerometer_top
- link fr3_hand: mass 0.73 -> 0.6544
- link fr3_leftfinger: mass 0.015 -> 0.0291
- link fr3_link0: geometry collision mesh filename=package://franka_description/meshes/robots/fr3/collision/li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; visual mesh filename=package://franka_description/meshes/robots/fr3/visual/link0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
- link fr3_link1: geometry collision mesh filename=package://franka_description/meshes/robots/fr3/collision/li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; visual mesh filename=package://franka_description/meshes/robots/fr3/visual/link1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
- link fr3_link2: geometry collision mesh filename=package://franka_description/meshes/robots/fr3/collision/li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; visual mesh filename=package://franka_description/meshes/robots/fr3/visual/link2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
- link fr3_link3: geometry collision mesh filename=package://franka_description/meshes/robots/fr3/collision/li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; visual mesh filename=package://franka_description/meshes/robots/fr3/visual/link3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
- link fr3_link4: geometry collision mesh filename=package://franka_description/meshes/robots/fr3/collision/li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; visual mesh filename=package://franka_description/meshes/robots/fr3/visual/link4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
- link fr3_link5: geometry collision mesh filename=package://franka_description/meshes/robots/fr3/collision/li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; visual mesh filename=package://franka_description/meshes/robots/fr3/visual/link5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
- link fr3_link6: geometry collision mesh filename=package://franka_description/meshes/robots/fr3/collision/li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; visual mesh filename=package://franka_description/meshes/robots/fr3/visual/link6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
- link fr3_link7: geometry collision mesh filename=package://franka_description/meshes/robots/fr3/collision/li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; visual mesh filename=package://franka_description/meshes/robots/fr3/visual/link7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
- link fr3_rightfinger: mass 0.015 -> 0.0291
Joints:
- added joint fr3_link0_accelerometer_bottom_joint: type fixed, parent fr3_link0, child fr3_link0_accelerometer_bottom, origin xyz=-0.019739 0.0015506 0.05075 rpy=0.0 0.0 -1.5708
- added joint fr3_link0_accelerometer_top_joint: type fixed, parent fr3_link0, child fr3_link0_accelerometer_top, origin xyz=-0.017402 -0.007872 0.04715 rpy=3.1416 0.0 0.0
- added joint fr3_link1_accelerometer_bottom_joint: type fixed, parent fr3_link1, child fr3_link1_accelerometer_bottom, origin xyz=0.01974 -0.08975 0.00155 rpy=-1.5708 1.5708 0.0
- added joint fr3_link1_accelerometer_top_joint: type fixed, parent fr3_link1, child fr3_link1_accelerometer_top, origin xyz=0.017402 -0.093352 -0.00787 rpy=-1.5708 0.0 3.1416
- added joint fr3_link2_accelerometer_bottom_joint: type fixed, parent fr3_link2, child fr3_link2_accelerometer_bottom, origin xyz=0.019737 -0.11875 -0.00155 rpy=1.5708 -1.5708 0.0
- added joint fr3_link2_accelerometer_top_joint: type fixed, parent fr3_link2, child fr3_link2_accelerometer_top, origin xyz=0.017403 -0.11715 0.00787 rpy=1.5708 0.0 3.1416
- added joint fr3_link3_accelerometer_bottom_joint: type fixed, parent fr3_link3, child fr3_link3_accelerometer_bottom, origin xyz=0.062769 0.073756 0.00155 rpy=1.5708 1.5708 0.0
- added joint fr3_link3_accelerometer_top_joint: type fixed, parent fr3_link3, child fr3_link3_accelerometer_top, origin xyz=0.065099 0.077352 -0.00787 rpy=-1.5708 0.0 0.0
- added joint fr3_link4_accelerometer_bottom_joint: type fixed, parent fr3_link4, child fr3_link4_accelerometer_bottom, origin xyz=-0.062775 0.049753 0.00155 rpy=-1.5708 1.5708 0.0
- added joint fr3_link4_accelerometer_top_joint: type fixed, parent fr3_link4, child fr3_link4_accelerometer_top, origin xyz=-0.0651 0.046252 -0.00787 rpy=-1.5708 0.0 -3.1416
- added joint fr3_link5_accelerometer_bottom_joint: type fixed, parent fr3_link5, child fr3_link5_accelerometer_bottom, origin xyz=-0.019742 0.082275 0.00146 rpy=1.5708 1.5708 0.0
- added joint fr3_link5_accelerometer_top_joint: type fixed, parent fr3_link5, child fr3_link5_accelerometer_top, origin xyz=-0.017363 0.085872 -0.00795 rpy=-1.5708 0.0 0.0
- joint fr3_finger_joint2: axis 0 -1 0 -> 0 1 0; origin xyz=0 0 0.0584 rpy=0 0 0 -> xyz=0 0 0.0584 rpy=0 0 3.141592653589793
- joint fr3_joint1: limit lower=-2.7437 upper=2.7437 effort=87.0 velocity=2.62 -> lower=-2.9007 upper=2.9007 effort=87.0 velocity=2.62
- joint fr3_joint2: limit lower=-1.7837 upper=1.7837 effort=87.0 velocity=2.62 -> lower=-1.8361 upper=1.8361 effort=87.0 velocity=2.62
- joint fr3_joint4: limit lower=-3.0421 upper=-0.1518 effort=87.0 velocity=2.62 -> lower=-3.077 upper=-0.1169 effort=87.0 velocity=2.62
- joint fr3_joint5: limit lower=-2.8065 upper=2.8065 effort=12.0 velocity=5.26 -> lower=-2.8763 upper=2.8763 effort=12.0 velocity=5.26
- joint fr3_joint6: limit lower=0.5445 upper=4.5169 effort=12.0 velocity=4.18 -> lower=0.4398 upper=4.6216 effort=12.0 velocity=4.18
- joint fr3_joint7: limit lower=-3.0159 upper=3.0159 effort=12.0 velocity=5.26 -> lower=-3.0508 upper=3.0508 effort=12.0 velocity=5.26
