Commit message: Redo moveit2 packages

File: franka_robot.urdf (robot description, URDF)
Before this commit: robot fr3, 26 links, 25 joints
Links:
- added link fr3_camera_link, mass 0.05; collision box size=0.03 0.03 0.03; visual box size=0.03 0.03 0.03
- added link fr3_camera_link_optical
Joints:
- added joint fr3_camera_joint: type fixed, parent fr3_link8, child fr3_camera_link, origin xyz=0.05 -0.05 0.05 rpy=1.5707963267948966 -1.5707963267948966 0
- added joint fr3_camera_optical_joint: type fixed, parent fr3_camera_link, child fr3_camera_link_optical, origin xyz=0 0 0 rpy=0 0 0

File: src/franka_moveit_config/config/fr3.urdf.xacro (robot description, xacro)
@@ -3,5 +3,5 @@
     <xacro:arg name="initial_positions_file" default="initial_positions.yaml" />
     <!-- Import fr3 urdf file -->
-    <xacro:include filename="$(find franka_description)/urdfs/fr3_franka_hand.urdf" />
+    <xacro:include filename="$(find franka_description)/robots/fr3/fr3.urdf.xacro" />
     <!-- Import control_xacro -->
     <xacro:include filename="fr3.ros2_control.xacro" />
